File: EnviroTron/hardware/EnviroTron.sch (EAGLE design)
At the start: 38 parts

Commit message: Added PI filter to create analog voltage rail. Increased mic amp gain. Replaced mic with lower noise device.
Parts:
- AMP: value MCP6002 -> OPAMP-OPA2376-MSOP8; device EnviroTron:MCP6002 -> EnviroTron:OPAMP-OPA2376-MSOP8; SPICEPREFIX (none) -> J
- C11: value 100n -> 10n
- COMMS: SPICEPREFIX (none) -> X
Changed lines of the file:
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@@
 <part name="R3" library="EnviroTron" deviceset="R-US_" device="R0603" value="68k"/>
 <part name="TEMP" library="EnviroTron" deviceset="SHT21" device=""/>
-<part name="COMMS" library="EnviroTron" deviceset="WEMOS-D1-MINI" device=""/>
+<part name="COMMS" library="EnviroTron" deviceset="WEMOS-D1-MINI" device="">
+<attribute name="SPICEPREFIX" value="X"/>
+</part>
 <part name="PRESS" library="EnviroTron" deviceset="LPS22HB" device=""/>
 <part name="C7" library="EnviroTron" deviceset="C-US" device="C0603" value="100n"/>
@@
 <part name="R10" library="EnviroTron" deviceset="R-US_" device="R0603" value="180k"/>
 <part name="R11" library="EnviroTron" deviceset="R-US_" device="R0603" value="10k"/>
-<part name="C11" library="EnviroTron" deviceset="C-US" device="C0603" value="100n"/>
+<part name="C11" library="EnviroTron" deviceset="C-US" device="C0603" value="10n"/>
 <part name="FRAME1" library="EnviroTron" deviceset="LETTER_L" device="">
 <attribute name="SECTION" value="Sensor Board"/>
@@
 <part name="C16" library="EnviroTron" deviceset="C-US" device="C0603" value="1u"/>
 <part name="C17" library="EnviroTron" deviceset="C-US" device="C0603" value="1u"/>
-<part name="AMP" library="EnviroTron" deviceset="MCP6002" device=""/>
+<part name="AMP" library="EnviroTron" deviceset="OPAMP" device="-MSOP8" technology="-OPA2376">
+<attribute name="SPICEPREFIX" value="J"/>
+</part>
 </parts>
 <sheets>
